Commit message: Change robot dimensions

File: description/gazebo_control.xacro (robot description, xacro)
@@ -6,6 +6,6 @@
             <left_joint>left_wheel_joint</left_joint>
             <right_joint>right_wheel_joint</right_joint>
-            <wheel_separation>0.35</wheel_separation>
-            <wheel_diameter>0.1</wheel_diameter>
+            <wheel_separation>0.373</wheel_separation>
+            <wheel_diameter>0.2</wheel_diameter>
             <!--  Limits -->
             <max_wheel_torque>200</max_wheel_torque>

File: description/lidar.xacro (robot description, xacro)
@@ -4,5 +4,5 @@
         <parent link="chassis"/>
         <child link="laser_frame"/>
-        <origin xyz="0.1 0 0.175" rpy="0 0 0"/>
+        <origin xyz="0.400 0 0.160" rpy="0 0 0"/>
     </joint>
     <link name="laser_frame">
@@ -37,5 +37,5 @@
                 </scan>
                 <range>
-                    <min>0.3</min>
+                    <min>0.5</min>
                     <max>12</max>
                 </range>

File: description/robot_core.xacro (robot description, xacro)
@@ -36,18 +36,18 @@
     <link name="chassis">
         <visual>
-            <origin xyz="0.15 0 0.075"/>
+            <origin xyz="0.254 0 0.0675"/>
             <geometry>
-                <box size="0.3 0.3 0.15"/>
+                <box size="0.508 0.323 0.135"/>
             </geometry>
             <material name="white"/>
         </visual>
         <collision>
-            <origin xyz="0.15 0 0.075"/>
+            <origin xyz="0.254 0 0.0675"/>
             <geometry>
-                <box size="0.3 0.3 0.15"/>
+                <box size="0.508 0.323 0.135"/>
             </geometry>
         </collision>
-        <xacro:inertial_box mass="0.5" x="0.3" y="0.3" z="0.15">
-            <origin xyz="0.15 0 0.075" rpy="0 0 0"/>
+        <xacro:inertial_box mass="5.0" x="0.508" y="0.323" z="0.135">
+            <origin xyz="0.254 0 0.0675" rpy="0 0 0"/>
         </xacro:inertial_box>
     </link>
@@ -59,5 +59,5 @@
         <parent link="base_link"/>
         <child link="left_wheel"/>
-        <origin xyz="0 0.175 0" rpy="-${pi/2} 0 0"/>
+        <origin xyz="0 0.1865 0" rpy="-${pi/2} 0 0"/>
         <axis xyz="0 0 1"/>
     </joint>
@@ -65,5 +65,5 @@
         <visual>
             <geometry>
-                <cylinder radius="0.05" length="0.04"/>
+                <cylinder radius="0.10" length="0.04"/>
             </geometry>
             <material name="blue"/>
@@ -71,8 +71,8 @@
         <collision>
             <geometry>
-                <cylinder radius="0.05" length="0.04"/>
+                <cylinder radius="0.10" length="0.04"/>
             </geometry>
         </collision>
-        <xacro:inertial_cylinder mass="0.1" length="0.04" radius="0.05">
+        <xacro:inertial_cylinder mass="1.0" length="0.04" radius="0.10">
             <origin xyz="0 0 0" rpy="0 0 0"/>
         </xacro:inertial_cylinder>
@@ -85,5 +85,5 @@
         <parent link="base_link"/>
         <child link="right_wheel"/>
-        <origin xyz="0 -0.175 0" rpy="${pi/2} 0 0"/>
+        <origin xyz="0 -0.1865 0" rpy="${pi/2} 0 0"/>
         <axis xyz="0 0 -1"/>
     </joint>
@@ -91,5 +91,5 @@
         <visual>
             <geometry>
-                <cylinder radius="0.05" length="0.04"/>
+                <cylinder radius="0.10" length="0.04"/>
             </geometry>
             <material name="blue"/>
@@ -97,8 +97,8 @@
         <collision>
             <geometry>
-                <cylinder radius="0.05" length="0.04"/>
+                <cylinder radius="0.10" length="0.04"/>
             </geometry>
         </collision>
-        <xacro:inertial_cylinder mass="0.1" length="0.04" radius="0.05">
+        <xacro:inertial_cylinder mass="1.0" length="0.04" radius="0.10">
             <origin xyz="0 0 0" rpy="0 0 0"/>
         </xacro:inertial_cylinder>
@@ -111,10 +111,10 @@
         <parent link="chassis"/>
         <child link="caster_wheel"/>
-        <origin xyz="0.24 0 0"/>
+        <origin xyz="0.400 0 0"/>
     </joint>
     <link name="caster_wheel">
         <visual>
             <geometry>
-                <sphere radius="0.05"/>
+                <sphere radius="0.10"/>
             </geometry>
             <material name="black"/>
@@ -122,8 +122,8 @@
         <collision>
             <geometry>
-                <sphere radius="0.05"/>
+                <sphere radius="0.10"/>
             </geometry>
         </collision>
-        <xacro:inertial_sphere mass="0.1" radius="0.05">
+        <xacro:inertial_sphere mass="0.1" radius="0.10">
             <origin xyz="0 0 0" rpy="0 0 0"/>
         </xacro:inertial_sphere>
